Commit message: [modify]fix lidar and tf from baselink to odom

File: src/pynqcar_model/description/gazebo_control.xacro (robot description, xacro)
@@ -2,10 +2,24 @@
 <robot xmlns:xacro="http://www.ros.org/wiki/xacro">
     <gazebo>
-            <plugin name="wheel_drive" filename="libgazebo_ros_planar_move.so">
-                <commandTopic>cmd_vel</commandTopic>
+            <plugin name="wheel_drive" filename="libgazebo_ros_planar_move.so"><!-- plugin for omnidirectional wheel-->
+                <commandTopic>cmd_vel</commandTopic> <!-- subscribe cmd_vel topic-->
                 <odometryTopic>odom</odometryTopic>
                 <odometryFrame>odom</odometryFrame>
                 <odometryRate>50.0</odometryRate>
                 <robotBaseFram>base_link</robotBaseFram>
+                <!-- wheel information-->
+                <!--reference https://gazebosim.org/api/gazebo/6.1/classignition_1_1gazebo_1_1systems_1_1MecanumDrive.html#details-->
+                <front_left_joint>left_front_wheel_joint</front_left_joint>
+                <front_right_joint>right_front_wheel_joint</front_right_joint>
+                <back_left_joint>left_back_wheel_joint</back_left_joint>
+                <back_right_joint>right_back_wheel_joint</back_right_joint>
+                <wheel_separation>"chassis_size_y</wheel_separation>
+                <!-- output -->
+                <odometry_frame>odom</odometry_frame>
+                <robot_base_frame>base_link</robot_base_frame>
+                <publish_odom>true</publish_odom>
+                <publish_odom_tf>true</publish_odom_tf>
+                <publish_weel_tf>true</publish_weel_tf>
+                <publishWheelJointState>true</publishWheelJointState>
             </plugin>
     </gazebo>

File: src/pynqcar_model/description/robot_core.xacro (robot description, xacro)
@@ -93,31 +93,4 @@
         mass="${wheel_mass}"
     />
-<!--
-    <joint name="left_front_wheel_joint" type="continuous">
-        <parent link="base_link"/>
-        <child link="left_front_wheel"/>
-        <origin xyz = "${chassis_size_x/4} ${chassis_size_y/2} 0" rpy="-${pi/2} 0 0"/>
-        <axis xyz="0 0 1"/>
-    </joint>
--->
-    <!-- LEFT FRONT WHEEL LINK -->
-<!--
-    <link name="left_front_wheel">
-        <visual>
-            <geometry>
-                <cylinder radius = "${wheel_radius}" length = "${wheel_length}"/>
-            </geometry>
-            <material name="black"/>
-        </visual>
-        <collision>
-            <geometry>
-                <cylinder radius = "${wheel_radius}" length = "${wheel_length}"/>
-            </geometry>
-        </collision>
-        <xacro:inertial_cylinder mass="0.1" radius = "${wheel_radius}" length = "${wheel_length}">
-            <origin xyz="0 0 0" rpy = "0 0 0" />
-        </xacro:inertial_cylinder>
-    </link>
--->
     <gazebo reference="left_front_wheel_link">
         <material>
@@ -135,28 +108,4 @@
         mass="${wheel_mass}"
     />
-<!--
-    <joint name="left_back_wheel_joint" type="continuous">
-        <parent link="base_link"/>
-        <child link="left_back_wheel"/>
-        <origin xyz = "-${chassis_size_x/4} ${chassis_size_y/2} 0" rpy="-${pi/2} 0 0"/>
-        <axis xyz="0 0 1"/>
-    </joint>
-    <link name="left_back_wheel">
-        <visual>
-            <geometry>
-                <cylinder radius = "${wheel_radius}" length = "${wheel_length}"/>
-            </geometry>
-            <material name="black"/>
-        </visual>
-        <collision>
-            <geometry>
-                <cylinder radius = "${wheel_radius}" length = "${wheel_length}"/>
-            </geometry>
-        </collision>
-        <xacro:inertial_cylinder mass="0.1" radius = "${wheel_radius}" length = "${wheel_length}">
-            <origin xyz="0 0 0" rpy = "0 0 0" />
-        </xacro:inertial_cylinder>
-    </link>
--->
     <gazebo reference="left_back_wheel_link">
         <material>
@@ -174,28 +123,4 @@
         mass="${wheel_mass}"
     />
-<!--
-    <joint name="right_front_wheel_joint" type="continuous">
-        <parent link="base_link"/>
-        <child link="right_front_wheel"/>
-        <origin xyz = "${chassis_size_x/4} -${chassis_size_y/2} 0" rpy="${pi/2} 0 0"/>
-        <axis xyz="0 0 -1"/>
-    </joint>
-    <link name="right_front_wheel">
-        <visual>
-            <geometry>
-                <cylinder radius = "${wheel_radius}" length = "${wheel_length}"/>
-            </geometry>
-            <material name="black"/>
-        </visual>
-        <collision>
-            <geometry>
-                <cylinder radius = "${wheel_radius}" length = "${wheel_length}"/>
-            </geometry>
-        </collision>
-        <xacro:inertial_cylinder mass="0.1" radius = "${wheel_radius}" length = "${wheel_length}">
-            <origin xyz="0 0 0" rpy = "0 0 0" />
-        </xacro:inertial_cylinder>
-    </link>
--->
     <gazebo reference="right_front_wheel_link">
         <material>
@@ -213,28 +138,4 @@
         mass="${wheel_mass}"
     />
-<!--
-    <joint name="right_back_wheel_joint" type="continuous">
-        <parent link="base_link"/>
-        <child link="right_back_wheel"/>
-        <origin xyz = "-${chassis_size_x/4} -${chassis_size_y/2} 0" rpy="${pi/2} 0 0"/>
-        <axis xyz="0 0 -1"/>
-    </joint>
-    <link name="right_back_wheel">
-        <visual>
-            <geometry>
-                <cylinder radius = "${wheel_radius}" length = "${wheel_length}"/>
-            </geometry>
-            <material name="black"/>
-        </visual>
-        <collision>
-            <geometry>
-                <cylinder radius = "${wheel_radius}" length = "${wheel_length}"/>
-            </geometry>
-        </collision>
-        <xacro:inertial_cylinder mass="0.1" radius = "${wheel_radius}" length = "${wheel_length}">
-            <origin xyz="0 0 0" rpy = "0 0 0" />
-        </xacro:inertial_cylinder>
-    </link>
--->
     <gazebo reference="right_back_wheel_link">
         <material>
@@ -272,5 +173,5 @@
     <!--lidar-->
     <xacro:lidar
-    joint_xyz = "-0.1 0 ${chassis_size_z + 0.02}"
+    joint_xyz = "-0.1 0 ${chassis_size_z + 0.1}"
     joint_rpy = "0 0 0"
     radius = "0.05"
