Commit message: [add]add four driving wheel

File: src/pynqcar_model/description/robot_core.xacro (robot description, xacro)
@@ -52,3 +52,95 @@
         </xacro:inertial_box>
     </link>
+    <!-- LEFT FRONT WHEEL LINK -->
+    <joint name="left_front_wheel_joint" type="continuous">
+        <parent link="base_link"/>
+        <child link="left_front_wheel"/>
+        <!--
+            cylinder is by defualt are oriented along the z-axis
+            we need out wheel to be oriented along the y-axis(base_link)
+        -->
+        <!-- 輪子約在車身1/4處-->
+        <origin xyz = "0.125 0.15 0" rpy="-${pi/2} 0 0"/>
+        <!--axis of rotation-->
+        <!--rotate around z axis of wheel, anti-clockwise=>positive (right hand rule) -->
+        <axis xyz="0 0 1"/>
+    </joint>
+    <!-- LEFT FRONT WHEEL LINK -->
+    <link name="left_front_wheel">
+        <visual>
+            <geometry>
+                <cylinder radius = "0.05" length = "0.04"/>
+            </geometry>
+            <material name="black"/>
+        </visual>
+    </link>
+    <!-- LEFT BACK WHEEL LINK -->
+    <joint name="left_back_wheel_joint" type="continuous">
+        <parent link="base_link"/>
+        <child link="left_back_wheel"/>
+        <!--
+            cylinder is by defualt are oriented along the z-axis
+            we need out wheel to be oriented along the y-axis(base_link)
+        -->
+        <!-- 輪子約在車身3/4處 車身左側-->
+        <origin xyz = "-0.125 0.15 0" rpy="-${pi/2} 0 0"/>
+        <!--axis of rotation-->
+        <!--rotate around z axis of wheel, anti-clockwise=>positive (right hand rule) -->
+        <axis xyz="0 0 1"/>
+    </joint>
+    <!-- LEFT BACK WHEEL LINK -->
+    <link name="left_back_wheel">
+        <visual>
+            <geometry>
+                <cylinder radius = "0.05" length = "0.04"/>
+            </geometry>
+            <material name="black"/>
+        </visual>
+    </link>
+    <!-- RIGHT FRONT WHEEL LINK -->
+    <joint name="right_front_wheel_joint" type="continuous">
+        <parent link="base_link"/>
+        <child link="right_front_wheel"/>
+        <!--
+            cylinder is by defualt are oriented along the z-axis
+            we need out wheel to be oriented along the y-axis(base_link)
+        -->
+        <!-- 輪子約在車身1/4處-->
+        <origin xyz = "0.125 -0.15 0" rpy="${pi/2} 0 0"/>
+        <!--axis of rotation-->
+        <!--rotate around z axis of wheel, anti-clockwise=>positive (right hand rule) -->
+        <axis xyz="0 0 -1"/>
+    </joint>
+    <!-- RIGH FRONT WHEEL LINK -->
+    <link name="right_front_wheel">
+        <visual>
+            <geometry>
+                <cylinder radius = "0.05" length = "0.04"/>
+            </geometry>
+            <material name="black"/>
+        </visual>
+    </link>
+    <!-- RIGHT BACK WHEEL LINK -->
+    <joint name="right_back_wheel_joint" type="continuous">
+        <parent link="base_link"/>
+        <child link="right_back_wheel"/>
+        <!--
+            cylinder is by defualt are oriented along the z-axis
+            we need out wheel to be oriented along the y-axis(base_link)
+        -->
+        <!-- 輪子約在車身3/4處 車身左側-->
+        <origin xyz = "-0.125 -0.15 0" rpy="${pi/2} 0 0"/>
+        <!--axis of rotation-->
+        <!--rotate around z axis of wheel, anti-clockwise=>positive (right hand rule) -->
+        <axis xyz="0 0 -1"/>
+    </joint>
+    <!-- RIGHT FRONT WHEEL LINK -->
+    <link name="right_back_wheel">
+        <visual>
+            <geometry>
+                <cylinder radius = "0.05" length = "0.04"/>
+            </geometry>
+            <material name="black"/>
+        </visual>
+    </link>
 </robot>

Commit message: [add] add variable to make it parameterized

File: src/pynqcar_model/description/robot_core.xacro (robot description, xacro)
@@ -23,5 +23,8 @@
     <!-- origin, size, mass of pynqcar chassis -->
     <xacro:property name="chassis_origin" value="0.25 0 0.1" />   <!--移動機殼 讓base_link在車身中央之底部 同樣地，chassis之origin也在底部 所以x跟z分別往前和往上移動size的一半-->
-    <xacro:property name="chassis_geometry" value="0.5 0.3 0.2" />  <!--大致估測整個機殼大小，我認為z方向應該不是重點-->
+    <xacro:property name="chassis_size_x" value="0.5"/>
+    <xacro:property name="chassis_size_y" value="0.3"/>
+    <xacro:property name="chassis_size_z" value="0.15"/>
+    <xacro:property name="chassis_geometry" value="${chassis_size_x} ${chassis_size_y} ${chassis_size_z}" />  <!--大致估測整個機殼大小，我認為z方向應該不是重點-->
     <xacro:property name="chassis_mass" value="0.5" />
     <xacro:property name="chassis_massx" value="0.3" />
@@ -52,4 +55,21 @@
         </xacro:inertial_box>
     </link>
+    <!--setting for pynqcar_wheel -->
+    <!-- ======================================================================= -->
+    <!--
+        pynqcar的base_link設定在車子的正中心，然後
+        pyncar共有四個輪子，分別有四個：左前輪 左後輪 右前輪 右後輪，預設他們的origin：
+        左前輪：base_link的y軸正方向(左)移動1/2個機殼y方向長度，其x正方向移動1/4個機殼x方向長度
+        左後輪：base_link的y軸正方向(左)移動1/2個機殼y方向長度，其x負方向移動1/4個機殼x方向長度
+        右前輪：base_link的y軸負方向(右)移動1/2個機殼y方向長度，其x正方向移動1/4個機殼x方向長度
+        右後輪：base_link的y軸負方向(右)移動1/2個機殼y方向長度，其x負方向移動1/4個機殼x方向長度
+        <xacro:property name="chassis_size_x" value="0.5"/>
+        <xacro:property name="chassis_size_y" value="0.3"/>
+        <xacro:property name="chassis_size_z" value="0.2"/>
+        輪子的長度、半徑未知，仍須測量
+    -->
+    <xacro:property name="wheel_radius" value="0.05"/>
+    <xacro:property name="wheel_length" value="0.04"/>
+    <!--======================================================================= -->
     <!-- LEFT FRONT WHEEL LINK -->
     <joint name="left_front_wheel_joint" type="continuous">
@@ -61,5 +81,5 @@
         -->
         <!-- 輪子約在車身1/4處-->
-        <origin xyz = "0.125 0.15 0" rpy="-${pi/2} 0 0"/>
+        <origin xyz = "${chassis_size_x/4} ${chassis_size_y/2} 0" rpy="-${pi/2} 0 0"/>
         <!--axis of rotation-->
         <!--rotate around z axis of wheel, anti-clockwise=>positive (right hand rule) -->
@@ -70,5 +90,5 @@
         <visual>
             <geometry>
-                <cylinder radius = "0.05" length = "0.04"/>
+                <cylinder radius = "${wheel_radius}" length = "${wheel_length}"/>
             </geometry>
             <material name="black"/>
@@ -84,5 +104,5 @@
         -->
         <!-- 輪子約在車身3/4處 車身左側-->
-        <origin xyz = "-0.125 0.15 0" rpy="-${pi/2} 0 0"/>
+        <origin xyz = "-${chassis_size_x/4} ${chassis_size_y/2} 0" rpy="-${pi/2} 0 0"/>
         <!--axis of rotation-->
         <!--rotate around z axis of wheel, anti-clockwise=>positive (right hand rule) -->
@@ -93,5 +113,5 @@
         <visual>
             <geometry>
-                <cylinder radius = "0.05" length = "0.04"/>
+                <cylinder radius = "${wheel_radius}" length = "${wheel_length}"/>
             </geometry>
             <material name="black"/>
@@ -106,6 +126,6 @@
             we need out wheel to be oriented along the y-axis(base_link)
         -->
-        <!-- 輪子約在車身1/4處-->
-        <origin xyz = "0.125 -0.15 0" rpy="${pi/2} 0 0"/>
+        <!-- 輪子約在車身1/4處 右側-->
+        <origin xyz = "${chassis_size_x/4} -${chassis_size_y/2} 0" rpy="${pi/2} 0 0"/>
         <!--axis of rotation-->
         <!--rotate around z axis of wheel, anti-clockwise=>positive (right hand rule) -->
@@ -116,5 +136,5 @@
         <visual>
             <geometry>
-                <cylinder radius = "0.05" length = "0.04"/>
+                <cylinder radius = "${wheel_radius}" length = "${wheel_length}"/>
             </geometry>
             <material name="black"/>
@@ -129,6 +149,6 @@
             we need out wheel to be oriented along the y-axis(base_link)
         -->
-        <!-- 輪子約在車身3/4處 車身左側-->
-        <origin xyz = "-0.125 -0.15 0" rpy="${pi/2} 0 0"/>
+        <!-- 輪子約在車身3/4處 車身右側-->
+        <origin xyz = "-${chassis_size_x/4} -${chassis_size_y/2} 0" rpy="${pi/2} 0 0"/>
         <!--axis of rotation-->
         <!--rotate around z axis of wheel, anti-clockwise=>positive (right hand rule) -->
@@ -139,8 +159,22 @@
         <visual>
             <geometry>
-                <cylinder radius = "0.05" length = "0.04"/>
+                <cylinder radius = "${wheel_radius}" length = "${wheel_length}"/>
             </geometry>
             <material name="black"/>
         </visual>
     </link>
+    <!-- cat head link-->
+    <joint name="cat_head_link_joint" type="fixed">
+        <parent link="base_link"/>
+        <child link="cat_head_link"/>
+        <origin xyz="0.25 0 0.03" rpy = "0 ${pi/2} 0"/>
+    </joint>
+    <link name="cat_head_link">
+        <visual>
+            <geometry>
+                <cylinder radius = "0.06" length = "0.01"/>
+            </geometry>
+            <material name="blue"/>
+        </visual>
+    </link>
 </robot>

Commit message: [add]create core urdf

File: src/pynqcar_model/description/robot_core.xacro (robot description, xacro)
@@ -28,5 +28,5 @@
     <xacro:property name="chassis_geometry" value="${chassis_size_x} ${chassis_size_y} ${chassis_size_z}" />  <!--大致估測整個機殼大小，我認為z方向應該不是重點-->
     <xacro:property name="chassis_mass" value="0.5" />
-    <xacro:property name="chassis_massx" value="0.3" />
+    <xacro:property name="chassis_massx" value="0.5" />
     <xacro:property name="chassis_massy" value="0.3" />
     <xacro:property name="chassis_massz" value="0.15" />
@@ -94,4 +94,12 @@
             <material name="black"/>
         </visual>
+        <collision>
+            <geometry>
+                <cylinder radius = "${wheel_radius}" length = "${wheel_length}"/>
+            </geometry>
+        </collision>
+        <xacro:inertial_cylinder mass="0.1" radius = "${wheel_radius}" length = "${wheel_length}">
+            <origin xyz="0 0 0" rpy = "0 0 0" />
+        </xacro:inertial_cylinder>
     </link>
     <!-- LEFT BACK WHEEL LINK -->
@@ -117,4 +125,12 @@
             <material name="black"/>
         </visual>
+        <collision>
+            <geometry>
+                <cylinder radius = "${wheel_radius}" length = "${wheel_length}"/>
+            </geometry>
+        </collision>
+        <xacro:inertial_cylinder mass="0.1" radius = "${wheel_radius}" length = "${wheel_length}">
+            <origin xyz="0 0 0" rpy = "0 0 0" />
+        </xacro:inertial_cylinder>
     </link>
     <!-- RIGHT FRONT WHEEL LINK -->
@@ -140,4 +156,12 @@
             <material name="black"/>
         </visual>
+        <collision>
+            <geometry>
+                <cylinder radius = "${wheel_radius}" length = "${wheel_length}"/>
+            </geometry>
+        </collision>
+        <xacro:inertial_cylinder mass="0.1" radius = "${wheel_radius}" length = "${wheel_length}">
+            <origin xyz="0 0 0" rpy = "0 0 0" />
+        </xacro:inertial_cylinder>
     </link>
     <!-- RIGHT BACK WHEEL LINK -->
@@ -163,4 +187,12 @@
             <material name="black"/>
         </visual>
+        <collision>
+            <geometry>
+                <cylinder radius = "${wheel_radius}" length = "${wheel_length}"/>
+            </geometry>
+        </collision>
+        <xacro:inertial_cylinder mass="0.1" radius = "${wheel_radius}" length = "${wheel_length}">
+            <origin xyz="0 0 0" rpy = "0 0 0" />
+        </xacro:inertial_cylinder>
     </link>
     <!-- cat head link-->
@@ -177,4 +209,12 @@
             <material name="blue"/>
         </visual>
+        <collision>
+            <geometry>
+                <cylinder radius = "0.06" length = "0.01"/>
+            </geometry>
+        </collision>
+        <xacro:inertial_cylinder mass="0.1" radius = "0.06" length = "0.01">
+            <origin xyz="0 0 0" rpy = "0 0 0" />
+        </xacro:inertial_cylinder>
     </link>
 </robot>

Commit message: [modify] show color in gazebo

File: src/pynqcar_model/description/robot_core.xacro (robot description, xacro)
@@ -55,4 +55,9 @@
         </xacro:inertial_box>
     </link>
+    <gazebo reference="chassis">
+        <material>
+            Gazebo/Orange
+        </material>
+    </gazebo>
     <!--setting for pynqcar_wheel -->
     <!-- ======================================================================= -->
@@ -103,4 +108,9 @@
         </xacro:inertial_cylinder>
     </link>
+    <gazebo reference="left_front_wheel">
+        <material>
+            Gazebo/Black
+        </material>
+    </gazebo>
     <!-- LEFT BACK WHEEL LINK -->
     <joint name="left_back_wheel_joint" type="continuous">
@@ -134,4 +144,9 @@
         </xacro:inertial_cylinder>
     </link>
+    <gazebo reference="left_back_wheel">
+        <material>
+            Gazebo/Black
+        </material>
+    </gazebo>
     <!-- RIGHT FRONT WHEEL LINK -->
     <joint name="right_front_wheel_joint" type="continuous">
@@ -165,4 +180,9 @@
         </xacro:inertial_cylinder>
     </link>
+    <gazebo reference="right_front_wheel">
+        <material>
+            Gazebo/Black
+        </material>
+    </gazebo>
     <!-- RIGHT BACK WHEEL LINK -->
     <joint name="right_back_wheel_joint" type="continuous">
@@ -196,4 +216,9 @@
         </xacro:inertial_cylinder>
     </link>
+    <gazebo reference="right_back_wheel">
+        <material>
+            Gazebo/Black
+        </material>
+    </gazebo>
     <!-- cat head link-->
     <joint name="cat_head_link_joint" type="fixed">
@@ -218,3 +243,8 @@
         </xacro:inertial_cylinder>
     </link>
+    <gazebo reference="cat_head_link">
+        <material>
+            Gazebo/Blue
+        </material>
+    </gazebo>
 </robot>

Commit message: [add(test)]add mecanum wheel urdf(not been test)

File: src/pynqcar_model/description/robot_core.xacro (robot description, xacro)
@@ -2,4 +2,5 @@
 <robot xmlns:xacro="http://www.ros.org/wiki/xacro" >
     <xacro:include filename="inertial_macros.xacro"/>
+    <xacro:include filename ="mech/mecanum_wheel.urdf.xacro"/>
     <!-- Color setting-->
     <material name="white">
@@ -76,20 +77,26 @@
     <xacro:property name="wheel_radius" value="0.05"/>
     <xacro:property name="wheel_length" value="0.04"/>
+    <xacro:property name="wheel_mass" value="0.6"/>
     <!--======================================================================= -->
     <!-- LEFT FRONT WHEEL LINK -->
+    <xacro:mecanum_wheel
+        side="left_front"
+        radius="${wheel_radius}"
+        width="${wheel_length}"
+        pos_x="${chassis_size_x/4}"
+        pos_y="${chassis_size_y/2}"
+        pos_z="0"
+        mass="${wheel_mass}"
+    />
+<!--
     <joint name="left_front_wheel_joint" type="continuous">
         <parent link="base_link"/>
         <child link="left_front_wheel"/>
-        <!--
-            cylinder is by defualt are oriented along the z-axis
-            we need out wheel to be oriented along the y-axis(base_link)
-        -->
-        <!-- 輪子約在車身1/4處-->
         <origin xyz = "${chassis_size_x/4} ${chassis_size_y/2} 0" rpy="-${pi/2} 0 0"/>
-        <!--axis of rotation-->
-        <!--rotate around z axis of wheel, anti-clockwise=>positive (right hand rule) -->
         <axis xyz="0 0 1"/>
     </joint>
+-->
     <!-- LEFT FRONT WHEEL LINK -->
+<!--
     <link name="left_front_wheel">
         <visual>
@@ -108,5 +115,6 @@
         </xacro:inertial_cylinder>
     </link>
-    <gazebo reference="left_front_wheel">
+-->
+    <gazebo reference="left_front_wheel_link">
         <material>
             Gazebo/Black
@@ -114,18 +122,20 @@
     </gazebo>
     <!-- LEFT BACK WHEEL LINK -->
+    <xacro:mecanum_wheel
+        side="left_back"
+        radius="${wheel_radius}"
+        width="${wheel_length}"
+        pos_x="-${chassis_size_x/4}"
+        pos_y="${chassis_size_y/2}"
+        pos_z="0"
+        mass="${wheel_mass}"
+    />
+<!--
     <joint name="left_back_wheel_joint" type="continuous">
         <parent link="base_link"/>
         <child link="left_back_wheel"/>
-        <!--
-            cylinder is by defualt are oriented along the z-axis
-            we need out wheel to be oriented along the y-axis(base_link)
-        -->
-        <!-- 輪子約在車身3/4處 車身左側-->
         <origin xyz = "-${chassis_size_x/4} ${chassis_size_y/2} 0" rpy="-${pi/2} 0 0"/>
-        <!--axis of rotation-->
-        <!--rotate around z axis of wheel, anti-clockwise=>positive (right hand rule) -->
         <axis xyz="0 0 1"/>
     </joint>
-    <!-- LEFT BACK WHEEL LINK -->
     <link name="left_back_wheel">
         <visual>
@@ -144,5 +154,6 @@
         </xacro:inertial_cylinder>
     </link>
-    <gazebo reference="left_back_wheel">
+-->
+    <gazebo reference="left_back_wheel_link">
         <material>
             Gazebo/Black
@@ -150,18 +161,20 @@
     </gazebo>
     <!-- RIGHT FRONT WHEEL LINK -->
+    <xacro:mecanum_wheel
+        side="right_front"
+        radius="${wheel_radius}"
+        width="${wheel_length}"
+        pos_x="${chassis_size_x/4}"
+        pos_y="-${chassis_size_y/2}"
+        pos_z="0"
+        mass="${wheel_mass}"
+    />
+<!--
     <joint name="right_front_wheel_joint" type="continuous">
         <parent link="base_link"/>
         <child link="right_front_wheel"/>
-        <!--
-            cylinder is by defualt are oriented along the z-axis
-            we need out wheel to be oriented along the y-axis(base_link)
-        -->
-        <!-- 輪子約在車身1/4處 右側-->
         <origin xyz = "${chassis_size_x/4} -${chassis_size_y/2} 0" rpy="${pi/2} 0 0"/>
-        <!--axis of rotation-->
-        <!--rotate around z axis of wheel, anti-clockwise=>positive (right hand rule) -->
         <axis xyz="0 0 -1"/>
     </joint>
-    <!-- RIGH FRONT WHEEL LINK -->
     <link name="right_front_wheel">
         <visual>
@@ -180,5 +193,6 @@
         </xacro:inertial_cylinder>
     </link>
-    <gazebo reference="right_front_wheel">
+-->
+    <gazebo reference="right_front_wheel_link">
         <material>
             Gazebo/Black
@@ -186,18 +200,20 @@
     </gazebo>
     <!-- RIGHT BACK WHEEL LINK -->
+    <xacro:mecanum_wheel
+        side="right_back"
+        radius="${wheel_radius}"
+        width="${wheel_length}"
+        pos_x="-${chassis_size_x/4}"
+        pos_y="-${chassis_size_y/2}"
+        pos_z="0"
+        mass="${wheel_mass}"
+    />
+<!--
     <joint name="right_back_wheel_joint" type="continuous">
         <parent link="base_link"/>
         <child link="right_back_wheel"/>
-        <!--
-            cylinder is by defualt are oriented along the z-axis
-            we need out wheel to be oriented along the y-axis(base_link)
-        -->
-        <!-- 輪子約在車身3/4處 車身右側-->
         <origin xyz = "-${chassis_size_x/4} -${chassis_size_y/2} 0" rpy="${pi/2} 0 0"/>
-        <!--axis of rotation-->
-        <!--rotate around z axis of wheel, anti-clockwise=>positive (right hand rule) -->
         <axis xyz="0 0 -1"/>
     </joint>
-    <!-- RIGHT FRONT WHEEL LINK -->
     <link name="right_back_wheel">
         <visual>
@@ -216,5 +232,6 @@
         </xacro:inertial_cylinder>
     </link>
-    <gazebo reference="right_back_wheel">
+-->
+    <gazebo reference="right_back_wheel_link">
         <material>
             Gazebo/Black

Commit message: [add] add lidar description and enable gazebo simulation

File: src/pynqcar_model/description/robot_core.xacro (robot description, xacro)
@@ -3,4 +3,5 @@
     <xacro:include filename="inertial_macros.xacro"/>
     <xacro:include filename ="mech/mecanum_wheel.urdf.xacro"/>
+    <xacro:include filename = "sensor/lidar.xacro"/>
     <!-- Color setting-->
     <material name="white">
@@ -15,4 +16,7 @@
     <material name="black">
         <color rgba="0 0 0 1"/>
+    </material>
+    <material name="red">
+        <color rgba="1 0 0 1"/>
     </material>
     <!-- BASE LINK -->
@@ -265,3 +269,13 @@
         </material>
     </gazebo>
+    <!--sensor-->
+    <!--lidar-->
+    <xacro:lidar
+    joint_xyz = "-0.1 0 ${chassis_size_z + 0.02}"
+    joint_rpy = "0 0 0"
+    radius = "0.05"
+    length = "0.04"
+    color = "red"
+    mass = "0.1"
+    />
 </robot>

Commit message: [add]Running lidar_slam on simulation

File: src/pynqcar_model/description/robot_core.xacro (robot description, xacro)
@@ -22,4 +22,12 @@
     <!-- BASE LINK -->
     <link name="base_link">
+    </link>
+    <!--BASE_FOOTPRINT LINK-->
+    <joint name="base_footprint_joint" type="fixed">
+        <parent link="base_link"/>
+        <child link="base_footprint"/>
+        <origin xyz="0 0 0" rpy="0 0 0"/>
+    </joint>
+    <link name="base_footprint">
     </link>
     <!-- CHASSIS LINK -->
